Commit message: movemaster_control: nodo controller_manager con JTC y JSB
Nuevo paquete movemaster_control, junto al plugin en
src/movemaster_ros/movemaster_ros/, que arranca el nodo controller_manager de
ros2_control (Jazzy) con MovemasterHardware, JointStateBroadcaster y
JointTrajectoryController, más robot_state_publisher, del que el
controller_manager lee /robot_description.

joints.json es la única fuente de las articulaciones: de él salen el URDF
(cadena provisional sin geometría, límites y velocidad máxima), el bloque
<ros2_control>, los joints del JTC y el update_rate (1/period_s).
use_mock_hardware:=true usa mock_components/GenericSystem sin CAN ni motores.

- config/ros2_control.xacro del plugin: genera las articulaciones desde
  joint_config_path (antes fijaba joint_1..3 y on_init rechazaba el
  joints.json actual de un eje) y admite use_mock_hardware.
- colcon_defaults.yaml: colcon no busca paquetes dentro del paquete Python
  movemaster_ros, así que se añade src/movemaster_ros/movemaster_ros como base.
- COLCON_IGNORE en src/movemaster_hardware: sin él, colcon compilaba esa
  versión anterior del plugin en lugar de la vigente.

Verificado sin ROS instalado: xacro 2.0.13 en modo real, simulado y con 3
ejes; pytest del paquete 6/6 (detecta 4 mutaciones); YAML contra las
definiciones de parámetros de Jazzy; lógica del launch con la librería launch
de Jazzy; load_driver_config y MoveMasterDriver aceptan el URDF generado;
colcon list/graph; flake8 con las reglas de ament.

Co-Authored-By: Claude Opus 5.5 <noreply@anthropic.com>
Claude-Session: https://claude.ai/code/session_01KU4gmWQbE5WkyeG6XjuBma

File: movemaster_ws/src/movemaster_ros/movemaster_ros/movemaster_hardware/config/ros2_control.xacro (robot description, xacro)
@@ -1,25 +1,45 @@
 <?xml version="1.0"?>
-<!-- Include this macro from your future robot URDF. It does not define geometry. -->
+<!-- Include this macro from the robot URDF. It does not define geometry.
+     The joints come from joint_config_path (joints.json), in file order, so the
+     ros2_control block always matches the joint list the plugin requires. -->
 <robot xmlns:xacro="http://www.ros.org/wiki/xacro">
-  <xacro:macro name="movemaster_control_joint" params="name">
+  <!-- initial_value is only read by mock hardware; MovemasterHardware reads the encoders. -->
+  <xacro:macro name="movemaster_control_joint" params="name initial_position:=0.0">
     <joint name="${name}">
       <command_interface name="position"/>
-      <state_interface name="position"/>
+      <state_interface name="position">
+        <param name="initial_value">${initial_position}</param>
+      </state_interface>
       <state_interface name="velocity"/>
       <state_interface name="current"/>
     </joint>
   </xacro:macro>
-  <xacro:macro name="movemaster_ros2_control" params="name spec_path joint_config_path can_interface:=can0">
+  <!-- One joint per entry of joints.json; mock hardware starts at 0 rad clamped to the limits. -->
+  <xacro:macro name="movemaster_control_joints" params="joints names">
+    <xacro:if value="${names}">
+      <xacro:property name="lower" value="${float(joints[names[0]]['min_position_rad'])}"/>
+      <xacro:property name="upper" value="${float(joints[names[0]]['max_position_rad'])}"/>
+      <xacro:movemaster_control_joint name="${names[0]}" initial_position="${min(max(0.0, lower), upper)}"/>
+      <xacro:movemaster_control_joints joints="${joints}" names="${names[1:]}"/>
+    </xacro:if>
+  </xacro:macro>
+  <!-- use_mock_hardware:=true swaps the plugin for mock_components/GenericSystem, with the
+       same interfaces, to run the controllers without CAN or motors. -->
+  <xacro:macro name="movemaster_ros2_control"
+               params="name spec_path joint_config_path can_interface:=can0 use_mock_hardware:=false">
+    <xacro:property name="joints" value="${xacro.load_yaml(joint_config_path)['joints']}"/>
     <ros2_control name="${name}" type="system">
       <hardware>
-        <plugin>movemaster_hardware/MovemasterHardware</plugin>
-        <param name="spec_path">${spec_path}</param>
-        <param name="joint_config_path">${joint_config_path}</param>
-        <param name="can_interface">${can_interface}</param>
+        <xacro:if value="${use_mock_hardware}">
+          <plugin>mock_components/GenericSystem</plugin>
+        </xacro:if>
+        <xacro:unless value="${use_mock_hardware}">
+          <plugin>movemaster_hardware/MovemasterHardware</plugin>
+          <param name="spec_path">${spec_path}</param>
+          <param name="joint_config_path">${joint_config_path}</param>
+          <param name="can_interface">${can_interface}</param>
+        </xacro:unless>
       </hardware>
-      <xacro:movemaster_control_joint name="joint_1"/>
-      <xacro:movemaster_control_joint name="joint_2"/>
-      <xacro:movemaster_control_joint name="joint_3"/>
-      <!-- Add joint_4..6 here and in your configuration when physically installed. -->
+      <xacro:movemaster_control_joints joints="${joints}" names="${list(joints)}"/>
     </ros2_control>
   </xacro:macro>

Commit message: movemaster_description: URDF del brazo desde la tabla Denavit-Hartenberg
Paquete nuevo con el modelo que usan el controller_manager, RViz y MoveIt:

- config/dh.yaml: tabla DH estándar de los cinco ejes, postura Home y radios
  de los eslabones.
- urdf/movemaster_arm.xacro: cada fila crea joint_i (giro θ en z), el eslabón
  <label>_link y joint_i_dh (Tz(d)·Tx(a)·Rx(α)) hasta dh_frame_i; el último
  marco es tool0. Los ejes que no están en joints.json quedan fijos en Home.
- urdf/movemaster.urdf.xacro: base, cadena DH y bloque <ros2_control> de los
  ejes de joints.json; rechaza ejes que no están en la tabla. preview:=true
  mueve los cinco ejes sin ros2_control.
- launch/display.launch.py y rviz/display.rviz: vista previa con sliders,
  arrancando en Home.
- test/test_description.py: cinemática directa del URDF contra el producto DH,
  Home en (0.160, 0, 0.255) m, ejes fijos y bloque <ros2_control>.

movemaster_control usa este URDF por defecto; se quita el modelo provisional y
sus pruebas pasan a movemaster_description. La macro ros2_control acepta
initial_positions y el hardware simulado arranca en Home: en 0 rad, con los
ejes 3-5 fijos en Home, la muñeca atraviesa la cintura.

MANUAL, DICCIONARIO y README: el paquete nuevo, la vista previa y la
calibración del cero (encender en Home con zero_offset_rad = ángulo Home).

Co-Authored-By: Claude Opus 5.5 <noreply@anthropic.com>
Claude-Session: https://claude.ai/code/session_01KU4gmWQbE5WkyeG6XjuBma

File: movemaster_ws/src/movemaster_ros/movemaster_ros/movemaster_hardware/config/ros2_control.xacro (robot description, xacro)
@@ -15,17 +15,22 @@
     </joint>
   </xacro:macro>
-  <!-- One joint per entry of joints.json; mock hardware starts at 0 rad clamped to the limits. -->
-  <xacro:macro name="movemaster_control_joints" params="joints names">
+  <!-- One joint per entry of joints.json. Mock hardware starts at initial_positions[joint],
+       0 rad if absent, clamped to the limits. -->
+  <xacro:macro name="movemaster_control_joints" params="joints names initial_positions">
     <xacro:if value="${names}">
       <xacro:property name="lower" value="${float(joints[names[0]]['min_position_rad'])}"/>
       <xacro:property name="upper" value="${float(joints[names[0]]['max_position_rad'])}"/>
-      <xacro:movemaster_control_joint name="${names[0]}" initial_position="${min(max(0.0, lower), upper)}"/>
-      <xacro:movemaster_control_joints joints="${joints}" names="${names[1:]}"/>
+      <xacro:property name="initial" value="${float(initial_positions.get(names[0], 0.0))}"/>
+      <xacro:movemaster_control_joint name="${names[0]}" initial_position="${min(max(initial, lower), upper)}"/>
+      <xacro:movemaster_control_joints joints="${joints}" names="${names[1:]}"
+          initial_positions="${initial_positions}"/>
     </xacro:if>
   </xacro:macro>
   <!-- use_mock_hardware:=true swaps the plugin for mock_components/GenericSystem, with the
-       same interfaces, to run the controllers without CAN or motors. -->
+       same interfaces, to run the controllers without CAN or motors. initial_positions maps
+       joint names to the radians the mock starts at. -->
   <xacro:macro name="movemaster_ros2_control"
-               params="name spec_path joint_config_path can_interface:=can0 use_mock_hardware:=false">
+               params="name spec_path joint_config_path can_interface:=can0 use_mock_hardware:=false
+                       initial_positions:=${dict()}">
     <xacro:property name="joints" value="${xacro.load_yaml(joint_config_path)['joints']}"/>
     <ros2_control name="${name}" type="system">
@@ -41,5 +46,6 @@
         </xacro:unless>
       </hardware>
-      <xacro:movemaster_control_joints joints="${joints}" names="${list(joints)}"/>
+      <xacro:movemaster_control_joints joints="${joints}" names="${list(joints)}"
+          initial_positions="${initial_positions}"/>
     </ros2_control>
   </xacro:macro>
